Commit message: add stiffness xacro

File: src/fishingrod_description/urdf/fishingrod.xacro (robot description, xacro)
@@ -51,9 +51,9 @@
     <limit effort="10" velocity="1.0" lower="-3.14" upper="3.14" />
     <axis xyz="0 0 1"/>
-    <gazebo>
+    <!-- <gazebo>
       <dynamics damping="0.1" friction="0.2"/>
       <spring_reference>0.0</spring_reference>
       <spring_stiffness>100.0</spring_stiffness>
-    </gazebo>
+    </gazebo> -->
   </joint>
   <!-- Link 1 -->
@@ -89,7 +89,7 @@
     <axis xyz="0 0 1"/>
     <gazebo>
-      <dynamics damping="0.1" friction="0.2"/>
+      <dynamics damping="0.0955" friction="4.3262"/>
       <spring_reference>0.0</spring_reference>
-      <spring_stiffness>100.0</spring_stiffness>
+      <spring_stiffness>4.3262</spring_stiffness>
     </gazebo>
   </joint>
@@ -126,8 +126,8 @@
   <axis xyz="0 0 1"/>
   <gazebo>
-    <dynamics damping="0.1" friction="0.2"/>
-    <spring_reference>0.0</spring_reference>
-      <spring_stiffness>100.0</spring_stiffness>
-  </gazebo>
+      <dynamics damping="0.082" friction="3.8263"/>
+      <spring_reference>0.0</spring_reference>
+      <spring_stiffness>3.8263</spring_stiffness>
+    </gazebo>
 </joint>
 <!-- Link 3 -->
@@ -163,8 +163,8 @@
   <axis xyz="0 0 1"/>
   <gazebo>
-    <dynamics damping="0.1" friction="0.2"/>
-    <spring_reference>0.0</spring_reference>
-      <spring_stiffness>100.0</spring_stiffness>
-  </gazebo>
+      <dynamics damping="0.0635" friction="3.355"/>
+      <spring_reference>0.0</spring_reference>
+      <spring_stiffness>3.355</spring_stiffness>
+    </gazebo>
 </joint>
 <!-- Link 4 -->
@@ -200,8 +200,8 @@
   <axis xyz="0 0 1"/>
   <gazebo>
-    <dynamics damping="0.1" friction="0.2"/>
-    <spring_reference>0.0</spring_reference>
-      <spring_stiffness>100.0</spring_stiffness>
-  </gazebo>
+      <dynamics damping="0.041" friction="2.1504"/>
+      <spring_reference>0.0</spring_reference>
+      <spring_stiffness>2.1504</spring_stiffness>
+    </gazebo>
 </joint>
 <!-- Link 5 -->
@@ -237,8 +237,8 @@
   <axis xyz="0 0 1"/>
   <gazebo>
-    <dynamics damping="0.1" friction="0.2"/>
-    <spring_reference>0.0</spring_reference>
-      <spring_stiffness>100.0</spring_stiffness>
-  </gazebo>
+      <dynamics damping="0.028" friction="1.4875"/>
+      <spring_reference>0.0</spring_reference>
+      <spring_stiffness>1.4875</spring_stiffness>
+    </gazebo>
 </joint>
 <!-- Link 6 -->
@@ -274,8 +274,8 @@
   <axis xyz="0 0 1"/>
   <gazebo>
-    <dynamics damping="0.1" friction="0.2"/>
-    <spring_reference>0.0</spring_reference>
-      <spring_stiffness>100.0</spring_stiffness>
-  </gazebo>
+      <dynamics damping="0.028" friction="1.4875"/>
+      <spring_reference>0.0</spring_reference>
+      <spring_stiffness>1.4875</spring_stiffness>
+    </gazebo>
 </joint>
 <!-- Link 7 -->
@@ -311,7 +311,7 @@
   <axis xyz="0 0 1"/>
   <gazebo>
-    <dynamics damping="0.1" friction="0.2"/>
-    <spring_reference>0.0</spring_reference>
-      <spring_stiffness>100.0</spring_stiffness>
+    <dynamics damping="0.028" friction="1.4875"/>
+    <spring_reference>0.0</spring_reference>
+    <spring_stiffness>1.4875</spring_stiffness>
   </gazebo>
 </joint>
@@ -348,8 +348,8 @@
   <axis xyz="0 0 1"/>
   <gazebo>
-    <dynamics damping="0.1" friction="0.2"/>
-    <spring_reference>0.0</spring_reference>
-      <spring_stiffness>100.0</spring_stiffness>
-  </gazebo>
+      <dynamics damping="0.028" friction="1.4875"/>
+      <spring_reference>0.0</spring_reference>
+      <spring_stiffness>1.4875</spring_stiffness>
+    </gazebo>
 </joint>
 <!-- Link 9 -->
@@ -385,8 +385,8 @@
   <axis xyz="0 0 1"/>
   <gazebo>
-    <dynamics damping="0.1" friction="0.2"/>
-    <spring_reference>0.0</spring_reference>
-      <spring_stiffness>100.0</spring_stiffness>
-  </gazebo>
+      <dynamics damping="0.021" friction="1.11"/>
+      <spring_reference>0.0</spring_reference>
+      <spring_stiffness>1.11</spring_stiffness>
+    </gazebo>
 </joint>
 <!-- Link 10 -->
@@ -422,7 +422,7 @@
   <axis xyz="0 0 1"/>
   <gazebo>
-    <dynamics damping="0.1" friction="0.2"/>
-    <spring_reference>0.0</spring_reference>
-      <spring_stiffness>100.0</spring_stiffness>
+    <dynamics damping="0.001" friction="0.505"/>
+    <spring_reference>0.0</spring_reference>
+    <spring_stiffness>0.505</spring_stiffness>
   </gazebo>
 </joint>
@@ -451,5 +451,5 @@
   </link>
 </xacro:macro>
-    <!-- Joint 12 -->
+<!-- Joint 12 -->
 <joint name="Joint_12" type="revolute">
   <parent link="Link_11"/>
@@ -459,7 +459,7 @@
   <axis xyz="0 0 1"/>
   <gazebo>
-    <dynamics damping="0.1" friction="0.2"/>
-    <spring_reference>0.0</spring_reference>
-      <spring_stiffness>100.0</spring_stiffness>
+    <dynamics damping="0.001" friction="0.4563"/>
+    <spring_reference>0.0</spring_reference>
+    <spring_stiffness>0.4563</spring_stiffness>
   </gazebo>
 </joint>
@@ -496,7 +496,7 @@
   <axis xyz="0 0 1"/>
   <gazebo>
-    <dynamics damping="0.1" friction="0.2"/>
-    <spring_reference>0.0</spring_reference>
-      <spring_stiffness>100.0</spring_stiffness>
+    <dynamics damping="0.0075" friction="0.3812"/>
+    <spring_reference>0.0</spring_reference>
+    <spring_stiffness>0.3812</spring_stiffness>
   </gazebo>
 </joint>
@@ -533,7 +533,7 @@
   <axis xyz="0 0 1"/>
   <gazebo>
-    <dynamics damping="0.1" friction="0.2"/>
-    <spring_reference>0.0</spring_reference>
-      <spring_stiffness>100.0</spring_stiffness>
+    <dynamics damping="0.01" friction="0.6750"/>
+    <spring_reference>0.0</spring_reference>
+    <spring_stiffness>0.6750</spring_stiffness>
   </gazebo>
 </joint>
@@ -570,7 +570,7 @@
   <axis xyz="0 0 1"/>
   <gazebo>
-    <dynamics damping="0.1" friction="0.2"/>
-    <spring_reference>0.0</spring_reference>
-      <spring_stiffness>100.0</spring_stiffness>
+    <dynamics damping="0.0085" friction="0.4588"/>
+    <spring_reference>0.0</spring_reference>
+    <spring_stiffness>0.4588</spring_stiffness>
   </gazebo>
 </joint>
@@ -607,7 +607,7 @@
   <axis xyz="0 0 1"/>
   <gazebo>
-    <dynamics damping="0.1" friction="0.2"/>
-    <spring_reference>0.0</spring_reference>
-      <spring_stiffness>100.0</spring_stiffness>
+    <dynamics damping="0.007" friction="0.3625"/>
+    <spring_reference>0.0</spring_reference>
+    <spring_stiffness>0.3625</spring_stiffness>
   </gazebo>
 </joint>
@@ -644,7 +644,7 @@
   <axis xyz="0 0 1"/>
   <gazebo>
-    <dynamics damping="0.1" friction="0.2"/>
-    <spring_reference>0.0</spring_reference>
-      <spring_stiffness>100.0</spring_stiffness>
+    <dynamics damping="0.006" friction="0.3625"/>
+    <spring_reference>0.0</spring_reference>
+    <spring_stiffness>0.3625</spring_stiffness>
   </gazebo>
 </joint>
@@ -718,7 +718,7 @@
   <axis xyz="0 0 1"/>
   <gazebo>
-    <dynamics damping="0.1" friction="0.2"/>
-    <spring_reference>0.0</spring_reference>
-      <spring_stiffness>100.0</spring_stiffness>
+    <dynamics damping="0.0045" friction="0.2663"/>
+    <spring_reference>0.0</spring_reference>
+    <spring_stiffness>0.2663</spring_stiffness>
   </gazebo>
 </joint>
@@ -755,7 +755,7 @@
   <axis xyz="0 0 1"/>
   <gazebo>
-    <dynamics damping="0.1" friction="0.2"/>
-    <spring_reference>0.0</spring_reference>
-      <spring_stiffness>100.0</spring_stiffness>
+    <dynamics damping="0.003" friction="0.2"/>
+    <spring_reference>0.0</spring_reference>
+    <spring_stiffness>0.2</spring_stiffness>
   </gazebo>
 </joint>
@@ -792,7 +792,7 @@
   <axis xyz="0 0 1"/>
   <gazebo>
-    <dynamics damping="0.1" friction="0.2"/>
-    <spring_reference>0.0</spring_reference>
-      <spring_stiffness>100.0</spring_stiffness>
+    <dynamics damping="0.002" friction="0.15"/>
+    <spring_reference>0.0</spring_reference>
+    <spring_stiffness>0.15</spring_stiffness>
   </gazebo>
 </joint>
