Commit message: urdf ros2_control

File: src/fishingrod_description/urdf/fishingrod.urdf (robot description, URDF)
Before this commit: robot fishingrod, 25 links, 24 joints
Joints:
- joint Joint_1: limit lower=-3.14 upper=3.14 effort=10 velocity=1.0 -> lower=-3.14 upper=3.14 effort=100 velocity=100.0

File: src/fishingrod_description/urdf/fishingrod.xacro (robot description, xacro)
@@ -49,5 +49,5 @@
     <child link="Link_1"/>
     <origin rpy="1.5708 0 0" xyz="0 0 0.09"/>
-    <limit effort="10" velocity="1.0" lower="-3.14" upper="3.14" />
+    <limit effort="100" velocity="100.0" lower="-3.14" upper="3.14" />
     <axis xyz="0 0 1"/>
     <!-- <gazebo>
